File: tools/r2r_dac/r2r_basys_DACs/r2r_basys_DACs.kicad_pcb (KiCad board)
At the start: 2 copper layers, 26.8 x 71.1 mm, 40 parts

Commit message: r2r dac + some fixes to final game - now it semiworks
Other:
- board text added: "uec2 mtm agh"
Changed lines of the file:
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@@
 		(allow_soldermask_bridges_in_footprints no)
 		(tenting front back)
+		(grid_origin 127 128.27)
 		(pcbplotparams
-			(layerselection 0x00000000_00000000_55555555_5755f5ff)
+			(layerselection 0x00000000_00000000_55555555_55555553)
 			(plot_on_all_layers_selection 0x00000000_00000000_00000000_00000000)
 			(disableapertmacros no)
@@
 			(crossoutdnponfab yes)
 			(subtractmaskfromsilk no)
-			(outputformat 1)
+			(outputformat 5)
 			(mirror no)
-			(drillshape 1)
+			(drillshape 0)
 			(scaleselection 1)
-			(outputdirectory "")
+			(outputdirectory "r2r_outputs/")
 		)
 	)
@@
 			)
 			(layer "F.SilkS")
-			(net 65793)
 		)
 		(fp_line
@@
 			)
 			(layer "F.SilkS")
-			(net 65793)
 		)
 		(fp_line
@@
 			)
 			(layer "F.SilkS")
-			(net 65793)
 		)
 		(fp_line
@@
 			)
 			(layer "F.SilkS")
-			(net 65793)
 		)
 		(fp_line
@@
 			)
 			(layer "F.CrtYd")
-			(net 65793)
 		)
 		(fp_line
@@
 			)
 			(layer "F.CrtYd")
-			(net 65793)
 		)
 		(fp_line
@@
 			)
 			(layer "F.CrtYd")
-			(net 65793)
 		)
 		(fp_line
@@
 			)
 			(layer "F.CrtYd")
-			(net 65793)
 		)
 		(pad "1" smd rect
@@
 	)
 	(gr_text "kszdomagh\n"
-		(at 152.273 104.521 90)
+		(at 151.892 125.857 90)
 		(layer "F.Cu" knockout)
 		(effects
@@
 		(layer "F.Cu" knockout)
 		(effects
+			(font
+				(size 1 1)
+				(thickness 0.2)
+				(bold yes)
+			)
+			(justify left bottom)
+		)
+	)
+	(gr_text "uec2 mtm agh"
+		(at 128.397 124.587 0)
+		(layer "F.Cu" knockout)
+		(effects
